File: soporoko.sch (KiCad schematic (older format))
At the start: 41 parts, among them P1 SWIM, P2 CAN, P3 CAN, P4 CONN_20X2, U1 LM7805CT, U2 STM8S208CBT, U3 MCP2551, X1 24MHz

Commit message: WIP: PCB
Parts:
- removed D1: LED, ~, symbol LED
- removed P2, P3: CAN, symbol CONN_4
- removed P4: CONN_20X2, symbol CONN_20X2
- removed R6: 1K, ~, symbol R
- added J1, J2: RJ45, symbol RJ45
- added P4, P5: CONN_6X2, symbol CONN_6X2
- added P7: CONN_4X2, symbol CONN_4X2
Connections:
- net C0: now also P7.1
- net C1: now also P7.3
- net C10: now also P5.1 (P1)
- net C11: now also P5.3 (P3)
- net C12: now also P5.5 (P5)
- net C13: now also P5.7 (P7)
- net C14: now also P5.9
- net C15: now also P5.11
- net C2: now also P7.5
- net C3: now also P7.7
- net C4: now also P4.1 (P1)
- net C5: now also P4.3 (P3)
- net C6: now also P4.5 (P5)
- net C7: now also P4.7 (P7)
- net C8: now also P4.9
- net C9: now also P4.11
- net CANH: now also J1.3, J2.3
- net CANL: now also J1.4, J2.4
- net GND: now also U1.2 (GND), J1.8, J2.8, P4.10, P4.12, P4.2 (P2), P4.4 (P4), P4.6 (P6), P4.8 (P8), P5.10, P5.12, P5.2 (P2), P5.4 (P4), P5.6 (P6), P5.8 (P8), P7.2, P7.4, P7.6, P7.8
- net V12: now also J1.1, J2.1
- net OUT0: no longer names the net of U2.44 (PD3)
- net OUT1: no longer names the net of U2.45 (PD4)
- net OUT2: no longer names the net of U2.46 (PD5)
- net OUT3: no longer names the net of U2.47 (PD6)
- net OUT4: no longer names the net of U2.48 (PD7)
- no-connect marks 13 -> 26
Other:
- moved on the sheet: JP1, R5
